File: nixie_clock/10hour.sch (KiCad schematic (older format))
At the start: 10 parts

Commit message: minor cleanups
Parts:
- removed C?: 0.1uF, symbol C
- removed P?: CONN_01X03, symbol CONN_01X03
- removed R?: 33K, symbol R
- removed R?: 1K, symbol R
- removed U? (x2): 4011, symbol 4011
- removed U?: IN-12, symbol IN-12
- added C5: 0.1uF, symbol C
- added P10: CONN_01X03, symbol CONN_01X03
- added R10: 33K, symbol R
- added R9: 1K, symbol R
- added U13: 4011, symbol 4011
- added U15: IN-12, symbol IN-12
- gave numbers to parts that had none: 3
Connections:
- net +220V: now also R10.2
- net +5V: now also R9.1, U13.14 (VDD), U13.14 (VDD)
- net CLK_IN: now also P10.3 (P3)
- net GND: now also U12.1 (CK), C5.2, U13.7 (VSS), U13.7 (VSS); no longer U12.9 (CK)
- net at U14.6 (INPUT_B): now also U12.4 (Q2), U13.1; no longer U12.12 (Q2)
- net at U14.3 (INPUT_A): now also U12.3 (Q1), U13.2; no longer U12.11 (Q1)
- net at U14.7 (INPUT_C): now also U12.5 (Q3); no longer U12.13 (Q3)
- net at U14.4 (INPUT_D): now also U12.6 (Q4); no longer U12.14 (Q4)
- net at U14.1 (OUT_8): now also U15.4 (8-KATOD)
- net at U14.10 (OUT_7): now also U15.5 (7-KATOD)
- net at U14.11 (OUT_6): now also U15.6 (6-KATOD)
- net at U14.13 (OUT_4): now also U15.8 (4-KATOD)
- net at U14.14 (OUT_5): now also U15.7 (5-KATOD)
- net at U14.15 (OUT_1): now also U15.11 (1-KATOD)
- net at U14.16 (OUT_0): now also U15.2 (0-KATOD)
- net at U14.2 (OUT_9): now also U15.3 (9-KATOD)
- net at U14.8 (OUT_2): now also U15.10 (2-KATOD)
- net at U14.9 (OUT_3): now also U15.9 (3-KATOD)
- net at P11.1 (P1): now also C5.1, P10.1 (P1), R9.2
- new net: P10.2 (P2), U12.2 (Enable)
- new net: U12.7 (Reset), U13.4
- new net: U13.3, U13.5, U13.6
- new net: R10.1, U15.1 (ANOD)

Commit message: Footprint associations
Parts:
- C5: footprint (none) -> Capacitors_THT:C_Axial_L5.1mm_D3.1mm_P7.50mm_Horizontal
- P10: footprint (none) -> Pin_Headers:Pin_Header_Straight_1x03_Pitch2.54mm
- P11: footprint (none) -> Pin_Headers:Pin_Header_Straight_1x02_Pitch2.54mm
- R10: footprint (none) -> hv:R_Axial_DIN0309_L9.0mm_D3.2mm_P12.70mm_Horizontal_Thick
- R9: footprint (none) -> Resistors_THT:R_Axial_DIN0207_L6.3mm_D2.5mm_P10.16mm_Horizontal
- U12, U14: footprint (none) -> Housings_DIP:DIP-16_W7.62mm
- U13: footprint (none) -> Housings_DIP:DIP-14_W7.62mm
- U15: footprint (none) -> hv:IN12
Changed lines of the file:
@@
 F 0 "U13" H 3900 3950 50  0000 C CNN
 F 1 "4011" H 3900 3850 50  0000 C CNN
-F 2 "" H 3900 3900 60  0001 C CNN
+F 2 "Housings_DIP:DIP-14_W7.62mm" H 3900 3900 60  0001 C CNN
 F 3 "" H 3900 3900 60  0001 C CNN
 	1    3900 3900
@@
 F 0 "U13" H 3950 4500 50  0000 C CNN
 F 1 "4011" H 3950 4400 50  0000 C CNN
-F 2 "" H 3950 4450 60  0001 C CNN
+F 2 "Housings_DIP:DIP-14_W7.62mm" H 3950 4450 60  0001 C CNN
 F 3 "" H 3950 4450 60  0001 C CNN
 	2    3950 4450
@@
 F 0 "U12" H 3950 3400 50  0000 C CNN
 F 1 "4518" H 4100 2600 50  0000 C CNN
-F 2 "" H 3900 2950 60  0001 C CNN
+F 2 "Housings_DIP:DIP-16_W7.62mm" H 3900 2950 60  0001 C CNN
 F 3 "" H 3900 2950 60  0001 C CNN
 	1    3900 2950
@@
 F 0 "U14" H 6800 3200 60  0000 C CNN
 F 1 "K155ID1" H 6850 3300 60  0000 C CNN
-F 2 "" H 6800 3350 60  0001 C CNN
+F 2 "Housings_DIP:DIP-16_W7.62mm" H 6800 3350 60  0001 C CNN
 F 3 "" H 6800 3350 60  0001 C CNN
 	1    6800 3350
@@
 F 0 "U15" H 9000 4650 60  0000 C CNN
 F 1 "IN-12" H 9000 4750 60  0000 C CNN
-F 2 "" H 9000 4750 60  0001 C CNN
+F 2 "hv:IN12" H 9000 4750 60  0001 C CNN
 F 3 "" H 9000 4750 60  0001 C CNN
 	1    9000 4750
@@
 F 0 "R10" V 8380 5900 50  0000 C CNN
 F 1 "33K" V 8300 5900 50  0000 C CNN
-F 2 "" V 8230 5900 50  0000 C CNN
+F 2 "hv:R_Axial_DIN0309_L9.0mm_D3.2mm_P12.70mm_Horizontal_Thick" V 8230 5900 50  0001 C CNN
 F 3 "" H 8300 5900 50  0000 C CNN
 	1    8300 5900
@@
 F 0 "P10" H 2200 3850 50  0000 C CNN
 F 1 "CONN_01X03" V 2300 3650 50  0000 C CNN
-F 2 "" H 2200 3650 50  0000 C CNN
+F 2 "Pin_Headers:Pin_Header_Straight_1x03_Pitch2.54mm" H 2200 3650 50  0001 C CNN
 F 3 "" H 2200 3650 50  0000 C CNN
 	1    2200 3650
@@
 F 0 "P11" H 2950 4000 50  0000 C CNN
 F 1 "CONN_01X02" V 3050 3850 50  0000 C CNN
-F 2 "" H 2950 3850 50  0000 C CNN
+F 2 "Pin_Headers:Pin_Header_Straight_1x02_Pitch2.54mm" H 2950 3850 50  0001 C CNN
 F 3 "" H 2950 3850 50  0000 C CNN
 	1    2950 3850
@@
 F 0 "R9" V 2530 3250 50  0000 C CNN
 F 1 "1K" V 2450 3250 50  0000 C CNN
-F 2 "" V 2380 3250 50  0000 C CNN
+F 2 "Resistors_THT:R_Axial_DIN0207_L6.3mm_D2.5mm_P10.16mm_Horizontal" V 2380 3250 50  0001 C CNN
 F 3 "" H 2450 3250 50  0000 C CNN
 	1    2450 3250
@@
 F 0 "C5" H 2625 3950 50  0000 L CNN
 F 1 "0.1uF" H 2400 3750 50  0000 L CNN
-F 2 "" H 2638 3700 50  0000 C CNN
+F 2 "Capacitors_THT:C_Axial_L5.1mm_D3.1mm_P7.50mm_Horizontal" H 2638 3700 50  0001 C CNN
 F 3 "" H 2600 3850 50  0000 C CNN
 	1    2600 3850
