File: nixie_clock/10minute.sch (KiCad schematic (older format))
At the start: 10 parts

Commit message: minor cleanups
Parts:
- removed C?: 0.1uF, symbol C
- removed P?: CONN_01X03, symbol CONN_01X03
- removed P?: CONN_01X02, symbol CONN_01X02
- removed R?: 33K, symbol R
- removed U?: 4518, symbol 4518
- removed U?: K155ID1, symbol K155ID1
- added C3: 0.1uF, symbol C
- added P6: CONN_01X03, symbol CONN_01X03
- added P7: CONN_01X02, symbol CONN_01X02
- added R6: 33K, symbol R
- added U7: 4518, symbol 4518
- added U8: K155ID1, symbol K155ID1
- gave numbers to parts that had none: 3
Connections:
- net +220V: now also R6.2
- net +5V: now also U7.16 (VDD), U8.5 (VCC)
- net CLK_IN: now also P6.3 (P3)
- net CLK_OUT: now also U7.5 (Q3), U8.7 (INPUT_C)
- net GND: now also C3.2, P7.2 (P2), U7.1 (CK), U7.8 (VSS), U8.12 (GND)
- net at U2.8: now also U7.4 (Q2), U8.6 (INPUT_B)
- net at U9.4 (8-KATOD): now also U8.1 (OUT_8)
- net at U9.5 (7-KATOD): now also U8.10 (OUT_7)
- net at U9.6 (6-KATOD): now also U8.11 (OUT_6)
- net at U9.8 (4-KATOD): now also U8.13 (OUT_4)
- net at U9.7 (5-KATOD): now also U8.14 (OUT_5)
- net at U9.11 (1-KATOD): now also U8.15 (OUT_1)
- net at U9.2 (0-KATOD): now also U8.16 (OUT_0)
- net at U9.3 (9-KATOD): now also U8.2 (OUT_9)
- net at U9.10 (2-KATOD): now also U8.8 (OUT_2)
- net at U9.9 (3-KATOD): now also U8.9 (OUT_3)
- net at U9.1 (ANOD): now also R6.1
- net at R5.2: now also C3.1, P6.1 (P1), P7.1 (P1)
- new net: U2.10, U2.12, U2.13
- new net: U2.11, U7.7 (Reset)
- new net: P6.2 (P2), U7.2 (Enable)
- new net: U7.3 (Q1), U8.3 (INPUT_A)
- new net: U7.6 (Q4), U8.4 (INPUT_D)

Commit message: Footprint associations
Parts:
- C3: footprint (none) -> Capacitors_THT:C_Axial_L5.1mm_D3.1mm_P7.50mm_Horizontal
- P6: footprint (none) -> Pin_Headers:Pin_Header_Straight_1x03_Pitch2.54mm
- P7: footprint (none) -> Pin_Headers:Pin_Header_Straight_1x02_Pitch2.54mm
- R5: footprint (none) -> Resistors_THT:R_Axial_DIN0207_L6.3mm_D2.5mm_P10.16mm_Horizontal
- R6: footprint (none) -> hv:R_Axial_DIN0309_L9.0mm_D3.2mm_P12.70mm_Horizontal_Thick
- U2: footprint (none) -> Housings_DIP:DIP-14_W7.62mm
- U7, U8: footprint (none) -> Housings_DIP:DIP-16_W7.62mm
- U9: footprint (none) -> hv:IN12
Changed lines of the file:
@@
 F 0 "U2" H 3900 3950 50  0000 C CNN
 F 1 "4011" H 3900 3850 50  0000 C CNN
-F 2 "" H 3900 3900 60  0001 C CNN
+F 2 "Housings_DIP:DIP-14_W7.62mm" H 3900 3900 60  0001 C CNN
 F 3 "" H 3900 3900 60  0001 C CNN
 	3    3900 3900
@@
 F 0 "U2" H 3950 4500 50  0000 C CNN
 F 1 "4011" H 3950 4400 50  0000 C CNN
-F 2 "" H 3950 4450 60  0001 C CNN
+F 2 "Housings_DIP:DIP-14_W7.62mm" H 3950 4450 60  0001 C CNN
 F 3 "" H 3950 4450 60  0001 C CNN
 	4    3950 4450
@@
 F 0 "U7" H 3950 3400 50  0000 C CNN
 F 1 "4518" H 4100 2600 50  0000 C CNN
-F 2 "" H 3900 2950 60  0001 C CNN
+F 2 "Housings_DIP:DIP-16_W7.62mm" H 3900 2950 60  0001 C CNN
 F 3 "" H 3900 2950 60  0001 C CNN
 	1    3900 2950
@@
 F 0 "U8" H 6800 3200 60  0000 C CNN
 F 1 "K155ID1" H 6850 3300 60  0000 C CNN
-F 2 "" H 6800 3350 60  0001 C CNN
+F 2 "Housings_DIP:DIP-16_W7.62mm" H 6800 3350 60  0001 C CNN
 F 3 "" H 6800 3350 60  0001 C CNN
 	1    6800 3350
@@
 F 0 "U9" H 9000 4650 60  0000 C CNN
 F 1 "IN-12" H 9000 4750 60  0000 C CNN
-F 2 "" H 9000 4750 60  0001 C CNN
+F 2 "hv:IN12" H 9000 4750 60  0001 C CNN
 F 3 "" H 9000 4750 60  0001 C CNN
 	1    9000 4750
@@
 F 0 "R6" V 8380 5900 50  0000 C CNN
 F 1 "33K" V 8300 5900 50  0000 C CNN
-F 2 "" V 8230 5900 50  0000 C CNN
+F 2 "hv:R_Axial_DIN0309_L9.0mm_D3.2mm_P12.70mm_Horizontal_Thick" V 8230 5900 50  0001 C CNN
 F 3 "" H 8300 5900 50  0000 C CNN
 	1    8300 5900
@@
 F 0 "P6" H 2200 3850 50  0000 C CNN
 F 1 "CONN_01X03" V 2300 3650 50  0000 C CNN
-F 2 "" H 2200 3650 50  0000 C CNN
+F 2 "Pin_Headers:Pin_Header_Straight_1x03_Pitch2.54mm" H 2200 3650 50  0001 C CNN
 F 3 "" H 2200 3650 50  0000 C CNN
 	1    2200 3650
@@
 F 0 "P7" H 2950 4000 50  0000 C CNN
 F 1 "CONN_01X02" V 3050 3850 50  0000 C CNN
-F 2 "" H 2950 3850 50  0000 C CNN
+F 2 "Pin_Headers:Pin_Header_Straight_1x02_Pitch2.54mm" H 2950 3850 50  0001 C CNN
 F 3 "" H 2950 3850 50  0000 C CNN
 	1    2950 3850
@@
 F 0 "R5" V 2530 3250 50  0000 C CNN
 F 1 "1K" V 2450 3250 50  0000 C CNN
-F 2 "" V 2380 3250 50  0000 C CNN
+F 2 "Resistors_THT:R_Axial_DIN0207_L6.3mm_D2.5mm_P10.16mm_Horizontal" V 2380 3250 50  0001 C CNN
 F 3 "" H 2450 3250 50  0000 C CNN
 	1    2450 3250
@@
 F 0 "C3" H 2625 3950 50  0000 L CNN
 F 1 "0.1uF" H 2400 3750 50  0000 L CNN
-F 2 "" H 2638 3700 50  0000 C CNN
+F 2 "Capacitors_THT:C_Axial_L5.1mm_D3.1mm_P7.50mm_Horizontal" H 2638 3700 50  0001 C CNN
 F 3 "" H 2600 3850 50  0000 C CNN
 	1    2600 3850
