File: nixie_clock/10second.sch (KiCad schematic (older format))
At the start: 10 parts

Commit message: minor cleanups
Parts:
- removed C?: 0.1uF, symbol C
- removed P?: CONN_01X03, symbol CONN_01X03
- removed P?: CONN_01X02, symbol CONN_01X02
- removed R?: 1K, symbol R
- removed U? (x2): 4011, symbol 4011
- removed U?: 4518, symbol 4518
- removed U?: K155ID1, symbol K155ID1
- removed U?: IN-12, symbol IN-12
- added C1: 0.1uF, symbol C
- added P2: CONN_01X03, symbol CONN_01X03
- added P3: CONN_01X02, symbol CONN_01X02
- added R1: 1K, symbol R
- added U1: 4518, symbol 4518
- added U2: 4011, symbol 4011
- added U3: K155ID1, symbol K155ID1
- added U4: IN-12, symbol IN-12
- gave numbers to parts that had none: 1
Connections:
- net +5V: now also R1.1, U1.16 (VDD), U2.14 (VDD), U2.14 (VDD), U3.5 (VCC)
- net CLK_IN: now also P2.3 (P3)
- net CLK_OUT: now also U1.5 (Q3), U2.2, U3.7 (INPUT_C)
- net GND: now also C1.2, P3.2 (P2), U1.1 (CK), U1.8 (VSS), U2.7 (VSS), U2.7 (VSS), U3.12 (GND)
- net at R2.1: now also U4.1 (ANOD)
- new net: U1.4 (Q2), U2.1, U3.6 (INPUT_B)
- new net: U2.3, U2.5, U2.6
- new net: U1.7 (Reset), U2.4
- new net: P2.2 (P2), U1.2 (Enable)
- new net: U1.3 (Q1), U3.3 (INPUT_A)
- new net: U1.6 (Q4), U3.4 (INPUT_D)
- new net: U3.1 (OUT_8), U4.4 (8-KATOD)
- new net: U3.10 (OUT_7), U4.5 (7-KATOD)
- new net: U3.11 (OUT_6), U4.6 (6-KATOD)
- new net: U3.13 (OUT_4), U4.8 (4-KATOD)
- new net: U3.14 (OUT_5), U4.7 (5-KATOD)
- new net: U3.15 (OUT_1), U4.11 (1-KATOD)
- new net: U3.16 (OUT_0), U4.2 (0-KATOD)
- new net: U3.2 (OUT_9), U4.3 (9-KATOD)
- new net: U3.8 (OUT_2), U4.10 (2-KATOD)
- new net: U3.9 (OUT_3), U4.9 (3-KATOD)
- new net: C1.1, P2.1 (P1), P3.1 (P1), R1.2

Commit message: Footprint associations
Parts:
- C1: footprint (none) -> Capacitors_THT:C_Axial_L5.1mm_D3.1mm_P7.50mm_Horizontal
- P2: footprint (none) -> Pin_Headers:Pin_Header_Straight_1x03_Pitch2.54mm
- P3: footprint (none) -> Pin_Headers:Pin_Header_Straight_1x02_Pitch2.54mm
- R1: footprint (none) -> Resistors_THT:R_Axial_DIN0207_L6.3mm_D2.5mm_P10.16mm_Horizontal
- R2: footprint (none) -> hv:R_Axial_DIN0309_L9.0mm_D3.2mm_P12.70mm_Horizontal_Thick
- U1, U3: footprint (none) -> Housings_DIP:DIP-16_W7.62mm
- U2: footprint (none) -> Housings_DIP:DIP-14_W7.62mm
- U4: footprint (none) -> hv:IN12
Changed lines of the file:
@@
 F 0 "U2" H 3900 3950 50  0000 C CNN
 F 1 "4011" H 3900 3850 50  0000 C CNN
-F 2 "" H 3900 3900 60  0001 C CNN
+F 2 "Housings_DIP:DIP-14_W7.62mm" H 3900 3900 60  0001 C CNN
 F 3 "" H 3900 3900 60  0001 C CNN
 	1    3900 3900
@@
 F 0 "U2" H 3950 4500 50  0000 C CNN
 F 1 "4011" H 3950 4400 50  0000 C CNN
-F 2 "" H 3950 4450 60  0001 C CNN
+F 2 "Housings_DIP:DIP-14_W7.62mm" H 3950 4450 60  0001 C CNN
 F 3 "" H 3950 4450 60  0001 C CNN
 	2    3950 4450
@@
 F 0 "U1" H 3950 3400 50  0000 C CNN
 F 1 "4518" H 4100 2600 50  0000 C CNN
-F 2 "" H 3900 2950 60  0001 C CNN
+F 2 "Housings_DIP:DIP-16_W7.62mm" H 3900 2950 60  0001 C CNN
 F 3 "" H 3900 2950 60  0001 C CNN
 	1    3900 2950
@@
 F 0 "U3" H 6800 3200 60  0000 C CNN
 F 1 "K155ID1" H 6850 3300 60  0000 C CNN
-F 2 "" H 6800 3350 60  0001 C CNN
+F 2 "Housings_DIP:DIP-16_W7.62mm" H 6800 3350 60  0001 C CNN
 F 3 "" H 6800 3350 60  0001 C CNN
 	1    6800 3350
@@
 F 0 "U4" H 9000 4650 60  0000 C CNN
 F 1 "IN-12" H 9000 4750 60  0000 C CNN
-F 2 "" H 9000 4750 60  0001 C CNN
+F 2 "hv:IN12" H 9000 4750 60  0001 C CNN
 F 3 "" H 9000 4750 60  0001 C CNN
 	1    9000 4750
@@
 F 0 "R2" V 8380 5900 50  0000 C CNN
 F 1 "33K" V 8300 5900 50  0000 C CNN
-F 2 "" V 8230 5900 50  0000 C CNN
+F 2 "hv:R_Axial_DIN0309_L9.0mm_D3.2mm_P12.70mm_Horizontal_Thick" V 8230 5900 50  0001 C CNN
 F 3 "" H 8300 5900 50  0000 C CNN
 	1    8300 5900
@@
 F 0 "P2" H 2200 3850 50  0000 C CNN
 F 1 "CONN_01X03" V 2300 3650 50  0000 C CNN
-F 2 "" H 2200 3650 50  0000 C CNN
+F 2 "Pin_Headers:Pin_Header_Straight_1x03_Pitch2.54mm" H 2200 3650 50  0001 C CNN
 F 3 "" H 2200 3650 50  0000 C CNN
 	1    2200 3650
@@
 F 0 "P3" H 2950 4000 50  0000 C CNN
 F 1 "CONN_01X02" V 3050 3850 50  0000 C CNN
-F 2 "" H 2950 3850 50  0000 C CNN
+F 2 "Pin_Headers:Pin_Header_Straight_1x02_Pitch2.54mm" H 2950 3850 50  0001 C CNN
 F 3 "" H 2950 3850 50  0000 C CNN
 	1    2950 3850
@@
 F 0 "R1" V 2530 3250 50  0000 C CNN
 F 1 "1K" V 2450 3250 50  0000 C CNN
-F 2 "" V 2380 3250 50  0000 C CNN
+F 2 "Resistors_THT:R_Axial_DIN0207_L6.3mm_D2.5mm_P10.16mm_Horizontal" V 2380 3250 50  0001 C CNN
 F 3 "" H 2450 3250 50  0000 C CNN
 	1    2450 3250
@@
 F 0 "C1" H 2625 3950 50  0000 L CNN
 F 1 "0.1uF" H 2400 3750 50  0000 L CNN
-F 2 "" H 2638 3700 50  0000 C CNN
+F 2 "Capacitors_THT:C_Axial_L5.1mm_D3.1mm_P7.50mm_Horizontal" H 2638 3700 50  0001 C CNN
 F 3 "" H 2600 3850 50  0000 C CNN
 	1    2600 3850
