File: nixie_clock/1hour.sch (KiCad schematic (older format))
At the start: 8 parts

Commit message: minor cleanups
Parts:
- removed C?: 0.1uF, symbol C
- removed P?: CONN_01X02, symbol CONN_01X02
- removed R?: 33K, symbol R
- removed R?: 1K, symbol R
- removed U?: 4518, symbol 4518
- removed U?: K155ID1, symbol K155ID1
- removed U?: IN-12, symbol IN-12
- added C4: 0.1uF, symbol C
- added P9: CONN_01X02, symbol CONN_01X02
- added R7: 1K, symbol R
- added R8: 33K, symbol R
- added U10: K155ID1, symbol K155ID1
- added U11: IN-12, symbol IN-12
- added U7: 4518, symbol 4518
- gave numbers to parts that had none: 1
Connections:
- net +220V: now also R8.2
- net +5V: now also R7.1, U10.5 (VCC), U7.16 (VDD)
- net CLK_OUT: now also U10.4 (INPUT_D), U7.14 (Q4)
- net GND: now also C4.2, P9.2 (P2), U10.12 (GND), U7.15 (Reset), U7.8 (VSS), U7.9 (CK)
- net at P8.2 (P2): now also U7.10 (Enable)
- net at P8.1 (P1): now also C4.1, P9.1 (P1), R7.2
- new net: U10.3 (INPUT_A), U7.11 (Q1)
- new net: U10.6 (INPUT_B), U7.12 (Q2)
- new net: U10.7 (INPUT_C), U7.13 (Q3)
- new net: U10.1 (OUT_8), U11.4 (8-KATOD)
- new net: U10.10 (OUT_7), U11.5 (7-KATOD)
- new net: U10.11 (OUT_6), U11.6 (6-KATOD)
- new net: U10.13 (OUT_4), U11.8 (4-KATOD)
- new net: U10.14 (OUT_5), U11.7 (5-KATOD)
- new net: U10.15 (OUT_1), U11.11 (1-KATOD)
- new net: U10.16 (OUT_0), U11.2 (0-KATOD)
- new net: U10.2 (OUT_9), U11.3 (9-KATOD)
- new net: U10.8 (OUT_2), U11.10 (2-KATOD)
- new net: U10.9 (OUT_3), U11.9 (3-KATOD)
- new net: R8.1, U11.1 (ANOD)
Changed lines of the file:
@@
 $EndDescr
 $Comp
-L 4518 U?
-U 1 1 590D5881
+L 4518 U7
+U 2 1 591359EA
 P 3900 2950
-F 0 "U?" H 3950 3400 50  0000 C CNN
+F 0 "U7" H 3950 3400 50  0000 C CNN
 F 1 "4518" H 4100 2600 50  0000 C CNN
 F 2 "" H 3900 2950 60  0001 C CNN
 F 3 "" H 3900 2950 60  0001 C CNN
-	1    3900 2950
-	1    0    0    -1
-$EndComp
-$Comp
-L K155ID1 U?
-U 1 1 590D5D46
+	2    3900 2950
+	1    0    0    -1
+$EndComp
+$Comp
+L K155ID1 U10
+U 1 1 591359EF
 P 6800 3350
-F 0 "U?" H 6800 3200 60  0000 C CNN
+F 0 "U10" H 6800 3200 60  0000 C CNN
 F 1 "K155ID1" H 6850 3300 60  0000 C CNN
 F 2 "" H 6800 3350 60  0001 C CNN
@@
 	5450 2600 4500 2600
 Wire Wire Line
-	6050 3300 5300 3300
-Wire Wire Line
-	5300 3300 4500 3300
+	4500 3300 6050 3300
 Wire Wire Line
 	4500 3300 4500 2900
@@
 	5050 3500 5050 3450
 $Comp
-L IN-12 U?
-U 1 1 590D638A
+L IN-12 U11
+U 1 1 591359F4
 P 9000 4750
-F 0 "U?" H 9000 4650 60  0000 C CNN
+F 0 "U11" H 9000 4650 60  0000 C CNN
 F 1 "IN-12" H 9000 4750 60  0000 C CNN
 F 2 "" H 9000 4750 60  0001 C CNN
@@
 $EndComp
 $Comp
-L R R?
-U 1 1 590D63EB
+L R R8
+U 1 1 591359F8
 P 8300 5900
-F 0 "R?" V 8380 5900 50  0000 C CNN
+F 0 "R8" V 8380 5900 50  0000 C CNN
 F 1 "33K" V 8300 5900 50  0000 C CNN
 F 2 "" V 8230 5900 50  0000 C CNN
@@
 NoConn ~ 9000 5750
 $Comp
-L +5V #PWR?
-U 1 1 590D6CDB
+L +5V #PWR064
+U 1 1 591359FC
 P 5700 2950
-F 0 "#PWR?" H 5700 2800 50  0001 C CNN
+F 0 "#PWR064" H 5700 2800 50  0001 C CNN
 F 1 "+5V" H 5700 3090 50  0000 C CNN
 F 2 "" H 5700 2950 50  0000 C CNN
@@
 $EndComp
 $Comp
-L GND #PWR?
-U 1 1 590D6CFB
+L GND #PWR065
+U 1 1 59135A02
 P 7550 3900
-F 0 "#PWR?" H 7550 3650 50  0001 C CNN
+F 0 "#PWR065" H 7550 3650 50  0001 C CNN
 F 1 "GND" H 7550 3750 50  0000 C CNN
 F 2 "" H 7550 3900 50  0000 C CNN
@@
 	7550 3900 7550 3400
 $Comp
-L +5V #PWR?
-U 1 1 590D72A1
-P 4800 1750
-F 0 "#PWR?" H 4800 1600 50  0001 C CNN
-F 1 "+5V" H 4800 1890 50  0000 C CNN
-F 2 "" H 4800 1750 50  0000 C CNN
-F 3 "" H 4800 1750 50  0000 C CNN
-	1    4800 1750
-	1    0    0    -1
-$EndComp
-$Comp
-L VDD #PWR?
+L +5V #PWR066
+U 1 1 59135A08
+P 4800 1700
+F 0 "#PWR066" H 4800 1550 50  0001 C CNN
+F 1 "+5V" H 4800 1840 50  0000 C CNN
+F 2 "" H 4800 1700 50  0000 C CNN
+F 3 "" H 4800 1700 50  0000 C CNN
+	1    4800 1700
+	1    0    0    -1
+$EndComp
+$Comp
+L VDD #PWR067
 U 1 1 590D72C1
-P 5100 1750
-F 0 "#PWR?" H 5100 1600 50  0001 C CNN
-F 1 "VDD" H 5100 1900 50  0000 C CNN
-F 2 "" H 5100 1750 50  0000 C CNN
-F 3 "" H 5100 1750 50  0000 C CNN
-	1    5100 1750
-	1    0    0    -1
-$EndComp
-$Comp
-L GND #PWR?
-U 1 1 590D72E1
-P 4800 2100
-F 0 "#PWR?" H 4800 1850 50  0001 C CNN
-F 1 "GND" H 4800 1950 50  0000 C CNN
-F 2 "" H 4800 2100 50  0000 C CNN
-F 3 "" H 4800 2100 50  0000 C CNN
-	1    4800 2100
-	1    0    0    -1
-$EndComp
-$Comp
-L VSS #PWR?
-U 1 1 590D7301
-P 5100 2100
-F 0 "#PWR?" H 5100 1950 50  0001 C CNN
-F 1 "VSS" H 5100 2250 50  0000 C CNN
-F 2 "" H 5100 2100 50  0000 C CNN
-F 3 "" H 5100 2100 50  0000 C CNN
-	1    5100 2100
+P 5100 1700
+F 0 "#PWR067" H 5100 1550 50  0001 C CNN
+F 1 "VDD" H 5100 1850 50  0000 C CNN
+F 2 "" H 5100 1700 50  0000 C CNN
+F 3 "" H 5100 1700 50  0000 C CNN
+	1    5100 1700
+	1    0    0    -1
+$EndComp
+$Comp
+L GND #PWR068
+U 1 1 59135A13
+P 4800 2150
+F 0 "#PWR068" H 4800 1900 50  0001 C CNN
+F 1 "GND" H 4800 2000 50  0000 C CNN
+F 2 "" H 4800 2150 50  0000 C CNN
+F 3 "" H 4800 2150 50  0000 C CNN
+	1    4800 2150
+	1    0    0    -1
+$EndComp
+$Comp
+L VSS #PWR069
+U 1 1 59135A18
+P 5100 2050
+F 0 "#PWR069" H 5100 1900 50  0001 C CNN
+F 1 "VSS" H 5100 2200 50  0000 C CNN
+F 2 "" H 5100 2050 50  0000 C CNN
+F 3 "" H 5100 2050 50  0000 C CNN
+	1    5100 2050
 	1    0    0    -1
 $EndComp
@@
 GND
 $Comp
-L +5V #PWR?
-U 1 1 590D7886
-P 2700 1950
-F 0 "#PWR?" H 2700 1800 50  0001 C CNN
-F 1 "+5V" H 2700 2090 50  0000 C CNN
-F 2 "" H 2700 1950 50  0000 C CNN
-F 3 "" H 2700 1950 50  0000 C CNN
-	1    2700 1950
-	1    0    0    -1
-$EndComp
-$Comp
-L GND #PWR?
+L +5V #PWR070
+U 1 1 59135A1A
+P 2700 1900
+F 0 "#PWR070" H 2700 1750 50  0001 C CNN
+F 1 "+5V" H 2700 2040 50  0000 C CNN
+F 2 "" H 2700 1900 50  0000 C CNN
+F 3 "" H 2700 1900 50  0000 C CNN
+	1    2700 1900
+	1    0    0    -1
+$EndComp
+$Comp
+L GND #PWR071
 U 1 1 590D78A6
-P 2700 2200
-F 0 "#PWR?" H 2700 1950 50  0001 C CNN
-F 1 "GND" H 2700 2050 50  0000 C CNN
-F 2 "" H 2700 2200 50  0000 C CNN
-F 3 "" H 2700 2200 50  0000 C CNN
-	1    2700 2200
+P 2700 2250
+F 0 "#PWR071" H 2700 2000 50  0001 C CNN
+F 1 "GND" H 2700 2100 50  0000 C CNN
+F 2 "" H 2700 2250 50  0000 C CNN
+F 3 "" H 2700 2250 50  0000 C CNN
+	1    2700 2250
 	1    0    0    -1
 $EndComp
@@
 	2600 1450 2700 1450
 $Comp
-L GND #PWR?
-U 1 1 590E0247
-P 2750 2800
-F 0 "#PWR?" H 2750 2550 50  0001 C CNN
-F 1 "GND" H 2750 2650 50  0000 C CNN
-F 2 "" H 2750 2800 50  0000 C CNN
-F 3 "" H 2750 2800 50  0000 C CNN
-	1    2750 2800
-	1    0    0    -1
-$EndComp
-Wire Wire Line
-	3300 2800 3000 2800
-Wire Wire Line
-	3000 2800 2750 2800
+L GND #PWR072
+U 1 1 59135A27
+P 2750 3100
+F 0 "#PWR072" H 2750 2850 50  0001 C CNN
+F 1 "GND" H 2750 2950 50  0000 C CNN
+F 2 "" H 2750 3100 50  0000 C CNN
+F 3 "" H 2750 3100 50  0000 C CNN
+	1    2750 3100
+	1    0    0    -1
+$EndComp
+Wire Wire Line
+	2750 2800 3300 2800
 Text HLabel 4750 3800 0    60   Input ~ 0
 CLK_OUT
@@
 	4750 3800 5300 3800
 $Comp
-L CONN_01X03 P?
+L CONN_01X03 P8
 U 1 1 590F618F
 P 2200 3650
-F 0 "P?" H 2200 3850 50  0000 C CNN
+F 0 "P8" H 2200 3850 50  0000 C CNN
 F 1 "CONN_01X03" V 2300 3650 50  0000 C CNN
 F 2 "" H 2200 3650 50  0000 C CNN
@@
 $EndComp
 $Comp
-L CONN_01X02 P?
-U 1 1 590F61CD
+L CONN_01X02 P9
+U 1 1 59135A2F
 P 2950 3850
-F 0 "P?" H 2950 4000 50  0000 C CNN
+F 0 "P9" H 2950 4000 50  0000 C CNN
 F 1 "CONN_01X02" V 3050 3850 50  0000 C CNN
 F 2 "" H 2950 3850 50  0000 C CNN
@@
 	2200 3000 3300 3000
 $Comp
-L R R?
-U 1 1 590F6393
+L R R7
+U 1 1 59135A34
 P 2450 3250
-F 0 "R?" V 2530 3250 50  0000 C CNN
+F 0 "R7" V 2530 3250 50  0000 C CNN
 F 1 "1K" V 2450 3250 50  0000 C CNN
 F 2 "" V 2380 3250 50  0000 C CNN
@@
 $EndComp
 $Comp
-L +5V #PWR?
-U 1 1 590F63C0
+L +5V #PWR073
+U 1 1 59135A3A
 P 2450 2950
-F 0 "#PWR?" H 2450 2800 50  0001 C CNN
+F 0 "#PWR073" H 2450 2800 50  0001 C CNN
 F 1 "+5V" H 2450 3090 50  0000 C CNN
 F 2 "" H 2450 2950 50  0000 C CNN
@@
 $EndComp
 $Comp
-L GND #PWR?
+L GND #PWR074
 U 1 1 590F63E6
 P 2750 4050
-F 0 "#PWR?" H 2750 3800 50  0001 C CNN
+F 0 "#PWR074" H 2750 3800 50  0001 C CNN
 F 1 "GND" H 2750 3900 50  0000 C CNN
 F 2 "" H 2750 4050 50  0000 C CNN
@@
 	2450 2950 2450 3100
 $Comp
-L C C?
-U 1 1 590F6DC1
+L C C4
+U 1 1 59135A41
 P 2600 3850
-F 0 "C?" H 2625 3950 50  0000 L CNN
+F 0 "C4" H 2625 3950 50  0000 L CNN
 F 1 "0.1uF" H 2400 3750 50  0000 L CNN
 F 2 "" H 2638 3700 50  0000 C CNN
@@
 $EndComp
 Wire Wire Line
-	2300 3450 2450 3450
-Wire Wire Line
-	2450 3450 2750 3450
-Wire Wire Line
-	2750 3450 2750 3700
-Wire Wire Line
-	2750 3700 2750 3800
-Wire Wire Line
-	2750 3900 2750 4000
-Wire Wire Line
-	2750 4000 2750 4050
+	2300 3450 2750 3450
+Wire Wire Line
+	2750 3450 2750 3800
+Wire Wire Line
+	2750 3900 2750 4050
 Wire Wire Line
 	2600 4000 2750 4000
@@
 Connection ~ 2450 3450
 $Comp
-L +220V #PWR?
-U 1 1 5910CD3A
-P 2700 1450
-F 0 "#PWR?" H 2700 1300 50  0001 C CNN
-F 1 "+220V" H 2700 1590 50  0000 C CNN
-F 2 "" H 2700 1450 50  0000 C CNN
-F 3 "" H 2700 1450 50  0000 C CNN
-	1    2700 1450
-	1    0    0    -1
-$EndComp
-$Comp
-L +220V #PWR?
+L +220V #PWR075
+U 1 1 59135A46
+P 2700 1400
+F 0 "#PWR075" H 2700 1250 50  0001 C CNN
+F 1 "+220V" H 2700 1540 50  0000 C CNN
+F 2 "" H 2700 1400 50  0000 C CNN
+F 3 "" H 2700 1400 50  0000 C CNN
+	1    2700 1400
+	1    0    0    -1
+$EndComp
+$Comp
+L +220V #PWR076
 U 1 1 5910CDE4
 P 7850 5850
-F 0 "#PWR?" H 7850 5700 50  0001 C CNN
+F 0 "#PWR076" H 7850 5700 50  0001 C CNN
 F 1 "+220V" H 7850 5990 50  0000 C CNN
 F 2 "" H 7850 5850 50  0000 C CNN
@@
 	5300 3800 5300 3300
 Connection ~ 5300 3300
+Wire Wire Line
+	5100 1750 5100 1700
+Wire Wire Line
+	5100 2100 5100 2050
+Wire Wire Line
+	4800 2150 4800 2100
+Wire Wire Line
+	4800 1750 4800 1700
+Wire Wire Line
+	2700 1450 2700 1400
+Wire Wire Line
+	2700 1950 2700 1900
+Wire Wire Line
+	2700 2250 2700 2200
+Wire Wire Line
+	2750 3100 2750 2800
 $EndSCHEMATC

Commit message: Footprint associations
Parts:
- C4: footprint (none) -> Capacitors_THT:C_Axial_L5.1mm_D3.1mm_P7.50mm_Horizontal
- P8: footprint (none) -> Pin_Headers:Pin_Header_Straight_1x03_Pitch2.54mm
- P9: footprint (none) -> Pin_Headers:Pin_Header_Straight_1x02_Pitch2.54mm
- R7: footprint (none) -> Resistors_THT:R_Axial_DIN0207_L6.3mm_D2.5mm_P10.16mm_Horizontal
- R8: footprint (none) -> hv:R_Axial_DIN0309_L9.0mm_D3.2mm_P12.70mm_Horizontal_Thick
- U10, U7: footprint (none) -> Housings_DIP:DIP-16_W7.62mm
- U11: footprint (none) -> hv:IN12
Changed lines of the file:
@@
 F 0 "U7" H 3950 3400 50  0000 C CNN
 F 1 "4518" H 4100 2600 50  0000 C CNN
-F 2 "" H 3900 2950 60  0001 C CNN
+F 2 "Housings_DIP:DIP-16_W7.62mm" H 3900 2950 60  0001 C CNN
 F 3 "" H 3900 2950 60  0001 C CNN
 	2    3900 2950
@@
 F 0 "U10" H 6800 3200 60  0000 C CNN
 F 1 "K155ID1" H 6850 3300 60  0000 C CNN
-F 2 "" H 6800 3350 60  0001 C CNN
+F 2 "Housings_DIP:DIP-16_W7.62mm" H 6800 3350 60  0001 C CNN
 F 3 "" H 6800 3350 60  0001 C CNN
 	1    6800 3350
@@
 F 0 "U11" H 9000 4650 60  0000 C CNN
 F 1 "IN-12" H 9000 4750 60  0000 C CNN
-F 2 "" H 9000 4750 60  0001 C CNN
+F 2 "hv:IN12" H 9000 4750 60  0001 C CNN
 F 3 "" H 9000 4750 60  0001 C CNN
 	1    9000 4750
@@
 F 0 "R8" V 8380 5900 50  0000 C CNN
 F 1 "33K" V 8300 5900 50  0000 C CNN
-F 2 "" V 8230 5900 50  0000 C CNN
+F 2 "hv:R_Axial_DIN0309_L9.0mm_D3.2mm_P12.70mm_Horizontal_Thick" V 8230 5900 50  0001 C CNN
 F 3 "" H 8300 5900 50  0000 C CNN
 	1    8300 5900
@@
 F 0 "P8" H 2200 3850 50  0000 C CNN
 F 1 "CONN_01X03" V 2300 3650 50  0000 C CNN
-F 2 "" H 2200 3650 50  0000 C CNN
+F 2 "Pin_Headers:Pin_Header_Straight_1x03_Pitch2.54mm" H 2200 3650 50  0001 C CNN
 F 3 "" H 2200 3650 50  0000 C CNN
 	1    2200 3650
@@
 F 0 "P9" H 2950 4000 50  0000 C CNN
 F 1 "CONN_01X02" V 3050 3850 50  0000 C CNN
-F 2 "" H 2950 3850 50  0000 C CNN
+F 2 "Pin_Headers:Pin_Header_Straight_1x02_Pitch2.54mm" H 2950 3850 50  0001 C CNN
 F 3 "" H 2950 3850 50  0000 C CNN
 	1    2950 3850
@@
 F 0 "R7" V 2530 3250 50  0000 C CNN
 F 1 "1K" V 2450 3250 50  0000 C CNN
-F 2 "" V 2380 3250 50  0000 C CNN
+F 2 "Resistors_THT:R_Axial_DIN0207_L6.3mm_D2.5mm_P10.16mm_Horizontal" V 2380 3250 50  0001 C CNN
 F 3 "" H 2450 3250 50  0000 C CNN
 	1    2450 3250
@@
 F 0 "C4" H 2625 3950 50  0000 L CNN
 F 1 "0.1uF" H 2400 3750 50  0000 L CNN
-F 2 "" H 2638 3700 50  0000 C CNN
+F 2 "Capacitors_THT:C_Axial_L5.1mm_D3.1mm_P7.50mm_Horizontal" H 2638 3700 50  0001 C CNN
 F 3 "" H 2600 3850 50  0000 C CNN
 	1    2600 3850
