File: nixie_clock/1minute.sch (KiCad schematic (older format))
At the start: 8 parts

Commit message: minor cleanups
Parts:
- removed P?: CONN_01X03, symbol CONN_01X03
- removed P?: CONN_01X02, symbol CONN_01X02
- removed R?: 33K, symbol R
- removed R?: 1K, symbol R
- removed U?: 4518, symbol 4518
- removed U?: K155ID1, symbol K155ID1
- removed U?: IN-12, symbol IN-12
- added P4: CONN_01X03, symbol CONN_01X03
- added P5: CONN_01X02, symbol CONN_01X02
- added R3: 1K, symbol R
- added R4: 33K, symbol R
- added U1: 4518, symbol 4518
- added U5: K155ID1, symbol K155ID1
- added U6: IN-12, symbol IN-12
- gave numbers to parts that had none: 1
Connections:
- net +220V: now also R4.2
- net +5V: now also R3.1, U1.16 (VDD), U5.5 (VCC)
- net CLK_IN: now also P4.3 (P3)
- net CLK_OUT: now also U1.14 (Q4), U5.4 (INPUT_D)
- net GND: now also P5.2 (P2), U1.15 (Reset), U1.8 (VSS), U1.9 (CK), U5.12 (GND)
- net at C2.1: now also P4.1 (P1), P5.1 (P1), R3.2
- new net: P4.2 (P2), U1.10 (Enable)
- new net: U1.11 (Q1), U5.3 (INPUT_A)
- new net: U1.12 (Q2), U5.6 (INPUT_B)
- new net: U1.13 (Q3), U5.7 (INPUT_C)
- new net: U5.1 (OUT_8), U6.4 (8-KATOD)
- new net: U5.10 (OUT_7), U6.5 (7-KATOD)
- new net: U5.11 (OUT_6), U6.6 (6-KATOD)
- new net: U5.13 (OUT_4), U6.8 (4-KATOD)
- new net: U5.14 (OUT_5), U6.7 (5-KATOD)
- new net: U5.15 (OUT_1), U6.11 (1-KATOD)
- new net: U5.16 (OUT_0), U6.2 (0-KATOD)
- new net: U5.2 (OUT_9), U6.3 (9-KATOD)
- new net: U5.8 (OUT_2), U6.10 (2-KATOD)
- new net: U5.9 (OUT_3), U6.9 (3-KATOD)
- new net: R4.1, U6.1 (ANOD)
Changed lines of the file:
@@
 $EndDescr
 $Comp
-L 4518 U?
-U 1 1 590D5881
+L 4518 U1
+U 2 1 591359EB
 P 3900 2950
-F 0 "U?" H 3950 3400 50  0000 C CNN
+F 0 "U1" H 3950 3400 50  0000 C CNN
 F 1 "4518" H 4100 2600 50  0000 C CNN
 F 2 "" H 3900 2950 60  0001 C CNN
 F 3 "" H 3900 2950 60  0001 C CNN
-	1    3900 2950
-	1    0    0    -1
-$EndComp
-$Comp
-L K155ID1 U?
-U 1 1 590D5D46
+	2    3900 2950
+	1    0    0    -1
+$EndComp
+$Comp
+L K155ID1 U5
+U 1 1 591359F0
 P 6800 3350
-F 0 "U?" H 6800 3200 60  0000 C CNN
+F 0 "U5" H 6800 3200 60  0000 C CNN
 F 1 "K155ID1" H 6850 3300 60  0000 C CNN
 F 2 "" H 6800 3350 60  0001 C CNN
@@
 	5450 2600 4500 2600
 Wire Wire Line
-	6050 3300 5300 3300
-Wire Wire Line
-	5300 3300 4500 3300
+	4500 3300 6050 3300
 Wire Wire Line
 	4500 3300 4500 2900
@@
 	5050 3500 5050 3450
 $Comp
-L IN-12 U?
-U 1 1 590D638A
+L IN-12 U6
+U 1 1 591359F1
 P 9000 4750
-F 0 "U?" H 9000 4650 60  0000 C CNN
+F 0 "U6" H 9000 4650 60  0000 C CNN
 F 1 "IN-12" H 9000 4750 60  0000 C CNN
 F 2 "" H 9000 4750 60  0001 C CNN
@@
 $EndComp
 $Comp
-L R R?
-U 1 1 590D63EB
+L R R4
+U 1 1 591359F7
 P 8300 5900
-F 0 "R?" V 8380 5900 50  0000 C CNN
+F 0 "R4" V 8380 5900 50  0000 C CNN
 F 1 "33K" V 8300 5900 50  0000 C CNN
 F 2 "" V 8230 5900 50  0000 C CNN
@@
 NoConn ~ 9000 5750
 $Comp
-L +5V #PWR?
+L +5V #PWR038
 U 1 1 590D6CDB
 P 5700 2950
-F 0 "#PWR?" H 5700 2800 50  0001 C CNN
+F 0 "#PWR038" H 5700 2800 50  0001 C CNN
 F 1 "+5V" H 5700 3090 50  0000 C CNN
 F 2 "" H 5700 2950 50  0000 C CNN
@@
 $EndComp
 $Comp
-L GND #PWR?
-U 1 1 590D6CFB
+L GND #PWR039
+U 1 1 59135A00
 P 7550 3900
-F 0 "#PWR?" H 7550 3650 50  0001 C CNN
+F 0 "#PWR039" H 7550 3650 50  0001 C CNN
 F 1 "GND" H 7550 3750 50  0000 C CNN
 F 2 "" H 7550 3900 50  0000 C CNN
@@
 	7550 3900 7550 3400
 $Comp
-L +5V #PWR?
-U 1 1 590D72A1
-P 4800 1750
-F 0 "#PWR?" H 4800 1600 50  0001 C CNN
-F 1 "+5V" H 4800 1890 50  0000 C CNN
-F 2 "" H 4800 1750 50  0000 C CNN
-F 3 "" H 4800 1750 50  0000 C CNN
-	1    4800 1750
-	1    0    0    -1
-$EndComp
-$Comp
-L VDD #PWR?
-U 1 1 590D72C1
-P 5100 1750
-F 0 "#PWR?" H 5100 1600 50  0001 C CNN
-F 1 "VDD" H 5100 1900 50  0000 C CNN
-F 2 "" H 5100 1750 50  0000 C CNN
-F 3 "" H 5100 1750 50  0000 C CNN
-	1    5100 1750
-	1    0    0    -1
-$EndComp
-$Comp
-L GND #PWR?
-U 1 1 590D72E1
-P 4800 2100
-F 0 "#PWR?" H 4800 1850 50  0001 C CNN
-F 1 "GND" H 4800 1950 50  0000 C CNN
-F 2 "" H 4800 2100 50  0000 C CNN
-F 3 "" H 4800 2100 50  0000 C CNN
-	1    4800 2100
-	1    0    0    -1
-$EndComp
-$Comp
-L VSS #PWR?
-U 1 1 590D7301
-P 5100 2100
-F 0 "#PWR?" H 5100 1950 50  0001 C CNN
-F 1 "VSS" H 5100 2250 50  0000 C CNN
-F 2 "" H 5100 2100 50  0000 C CNN
-F 3 "" H 5100 2100 50  0000 C CNN
-	1    5100 2100
+L +5V #PWR040
+U 1 1 59135A07
+P 4800 1700
+F 0 "#PWR040" H 4800 1550 50  0001 C CNN
+F 1 "+5V" H 4800 1840 50  0000 C CNN
+F 2 "" H 4800 1700 50  0000 C CNN
+F 3 "" H 4800 1700 50  0000 C CNN
+	1    4800 1700
+	1    0    0    -1
+$EndComp
+$Comp
+L VDD #PWR041
+U 1 1 59135A0C
+P 5100 1700
+F 0 "#PWR041" H 5100 1550 50  0001 C CNN
+F 1 "VDD" H 5100 1850 50  0000 C CNN
+F 2 "" H 5100 1700 50  0000 C CNN
+F 3 "" H 5100 1700 50  0000 C CNN
+	1    5100 1700
+	1    0    0    -1
+$EndComp
+$Comp
+L GND #PWR042
+U 1 1 59135A12
+P 4800 2150
+F 0 "#PWR042" H 4800 1900 50  0001 C CNN
+F 1 "GND" H 4800 2000 50  0000 C CNN
+F 2 "" H 4800 2150 50  0000 C CNN
+F 3 "" H 4800 2150 50  0000 C CNN
+	1    4800 2150
+	1    0    0    -1
+$EndComp
+$Comp
+L VSS #PWR043
+U 1 1 59135A14
+P 5100 2050
+F 0 "#PWR043" H 5100 1900 50  0001 C CNN
+F 1 "VSS" H 5100 2200 50  0000 C CNN
+F 2 "" H 5100 2050 50  0000 C CNN
+F 3 "" H 5100 2050 50  0000 C CNN
+	1    5100 2050
 	1    0    0    -1
 $EndComp
@@
 GND
 $Comp
-L +5V #PWR?
+L +5V #PWR044
 U 1 1 590D7886
-P 2700 1950
-F 0 "#PWR?" H 2700 1800 50  0001 C CNN
-F 1 "+5V" H 2700 2090 50  0000 C CNN
-F 2 "" H 2700 1950 50  0000 C CNN
-F 3 "" H 2700 1950 50  0000 C CNN
-	1    2700 1950
-	1    0    0    -1
-$EndComp
-$Comp
-L GND #PWR?
-U 1 1 590D78A6
-P 2700 2200
-F 0 "#PWR?" H 2700 1950 50  0001 C CNN
-F 1 "GND" H 2700 2050 50  0000 C CNN
-F 2 "" H 2700 2200 50  0000 C CNN
-F 3 "" H 2700 2200 50  0000 C CNN
-	1    2700 2200
+P 2700 1900
+F 0 "#PWR044" H 2700 1750 50  0001 C CNN
+F 1 "+5V" H 2700 2040 50  0000 C CNN
+F 2 "" H 2700 1900 50  0000 C CNN
+F 3 "" H 2700 1900 50  0000 C CNN
+	1    2700 1900
+	1    0    0    -1
+$EndComp
+$Comp
+L GND #PWR045
+U 1 1 59135A22
+P 2750 2250
+F 0 "#PWR045" H 2750 2000 50  0001 C CNN
+F 1 "GND" H 2750 2100 50  0000 C CNN
+F 2 "" H 2750 2250 50  0000 C CNN
+F 3 "" H 2750 2250 50  0000 C CNN
+	1    2750 2250
 	1    0    0    -1
 $EndComp
 Wire Wire Line
 	2600 1950 2700 1950
-Wire Wire Line
-	2700 2200 2600 2200
 Text HLabel 2600 1450 0    60   Input ~ 0
 220V
@@
 	2600 1450 2700 1450
 $Comp
-L GND #PWR?
+L GND #PWR046
 U 1 1 590E0247
-P 2750 2800
-F 0 "#PWR?" H 2750 2550 50  0001 C CNN
-F 1 "GND" H 2750 2650 50  0000 C CNN
-F 2 "" H 2750 2800 50  0000 C CNN
-F 3 "" H 2750 2800 50  0000 C CNN
-	1    2750 2800
-	1    0    0    -1
-$EndComp
-Wire Wire Line
-	3300 2800 3000 2800
-Wire Wire Line
-	3000 2800 2750 2800
+P 2900 3100
+F 0 "#PWR046" H 2900 2850 50  0001 C CNN
+F 1 "GND" H 2900 2950 50  0000 C CNN
+F 2 "" H 2900 3100 50  0000 C CNN
+F 3 "" H 2900 3100 50  0000 C CNN
+	1    2900 3100
+	1    0    0    -1
+$EndComp
 Text HLabel 4750 3800 0    60   Input ~ 0
 CLK_OUT
@@
 	4750 3800 5300 3800
 $Comp
-L CONN_01X03 P?
-U 1 1 590F618F
+L CONN_01X03 P4
+U 1 1 59135A2C
 P 2200 3650
-F 0 "P?" H 2200 3850 50  0000 C CNN
+F 0 "P4" H 2200 3850 50  0000 C CNN
 F 1 "CONN_01X03" V 2300 3650 50  0000 C CNN
 F 2 "" H 2200 3650 50  0000 C CNN
@@
 $EndComp
 $Comp
-L CONN_01X02 P?
-U 1 1 590F61CD
+L CONN_01X02 P5
+U 1 1 59135A2E
 P 2950 3850
-F 0 "P?" H 2950 4000 50  0000 C CNN
+F 0 "P5" H 2950 4000 50  0000 C CNN
 F 1 "CONN_01X02" V 3050 3850 50  0000 C CNN
 F 2 "" H 2950 3850 50  0000 C CNN
@@
 	2200 3000 3300 3000
 $Comp
-L R R?
-U 1 1 590F6393
+L R R3
+U 1 1 59135A36
 P 2450 3250
-F 0 "R?" V 2530 3250 50  0000 C CNN
+F 0 "R3" V 2530 3250 50  0000 C CNN
 F 1 "1K" V 2450 3250 50  0000 C CNN
 F 2 "" V 2380 3250 50  0000 C CNN
@@
 $EndComp
 $Comp
-L +5V #PWR?
-U 1 1 590F63C0
+L +5V #PWR047
+U 1 1 59135A39
 P 2450 2950
-F 0 "#PWR?" H 2450 2800 50  0001 C CNN
+F 0 "#PWR047" H 2450 2800 50  0001 C CNN
 F 1 "+5V" H 2450 3090 50  0000 C CNN
 F 2 "" H 2450 2950 50  0000 C CNN
@@
 $EndComp
 $Comp
-L GND #PWR?
-U 1 1 590F63E6
+L GND #PWR048
+U 1 1 59135A3D
 P 2750 4050
-F 0 "#PWR?" H 2750 3800 50  0001 C CNN
+F 0 "#PWR048" H 2750 3800 50  0001 C CNN
 F 1 "GND" H 2750 3900 50  0000 C CNN
 F 2 "" H 2750 4050 50  0000 C CNN
@@
 	2450 2950 2450 3100
 $Comp
-L C C?
+L C C2
 U 1 1 590F6DC1
 P 2600 3850
-F 0 "C?" H 2625 3950 50  0000 L CNN
+F 0 "C2" H 2625 3950 50  0000 L CNN
 F 1 "0.1uF" H 2400 3750 50  0000 L CNN
 F 2 "" H 2638 3700 50  0000 C CNN
@@
 $EndComp
 Wire Wire Line
-	2300 3450 2450 3450
-Wire Wire Line
-	2450 3450 2750 3450
-Wire Wire Line
-	2750 3450 2750 3700
-Wire Wire Line
-	2750 3700 2750 3800
-Wire Wire Line
-	2750 3900 2750 4000
-Wire Wire Line
-	2750 4000 2750 4050
+	2300 3450 2750 3450
+Wire Wire Line
+	2750 3450 2750 3800
+Wire Wire Line
+	2750 3900 2750 4050
 Wire Wire Line
 	2600 4000 2750 4000
@@
 Connection ~ 2450 3450
 $Comp
-L +220V #PWR?
-U 1 1 5910CD3A
-P 2700 1450
-F 0 "#PWR?" H 2700 1300 50  0001 C CNN
-F 1 "+220V" H 2700 1590 50  0000 C CNN
-F 2 "" H 2700 1450 50  0000 C CNN
-F 3 "" H 2700 1450 50  0000 C CNN
-	1    2700 1450
-	1    0    0    -1
-$EndComp
-$Comp
-L +220V #PWR?
-U 1 1 5910CDE4
+L +220V #PWR049
+U 1 1 59135A48
+P 2700 1400
+F 0 "#PWR049" H 2700 1250 50  0001 C CNN
+F 1 "+220V" H 2700 1540 50  0000 C CNN
+F 2 "" H 2700 1400 50  0000 C CNN
+F 3 "" H 2700 1400 50  0000 C CNN
+	1    2700 1400
+	1    0    0    -1
+$EndComp
+$Comp
+L +220V #PWR050
+U 1 1 59135A4D
 P 7850 5850
-F 0 "#PWR?" H 7850 5700 50  0001 C CNN
+F 0 "#PWR050" H 7850 5700 50  0001 C CNN
 F 1 "+220V" H 7850 5990 50  0000 C CNN
 F 2 "" H 7850 5850 50  0000 C CNN
@@
 	5300 3800 5300 3300
 Connection ~ 5300 3300
+Wire Wire Line
+	2900 3100 2900 2800
+Wire Wire Line
+	2900 2800 3300 2800
+Wire Wire Line
+	2600 2200 2750 2200
+Wire Wire Line
+	2750 2200 2750 2250
+Wire Wire Line
+	4800 2150 4800 2100
+Wire Wire Line
+	5100 1700 5100 1750
+Wire Wire Line
+	5100 2100 5100 2050
+Wire Wire Line
+	4800 1750 4800 1700
+Wire Wire Line
+	2700 1450 2700 1400
+Wire Wire Line
+	2700 1950 2700 1900
 $EndSCHEMATC

Commit message: Footprint associations
Parts:
- C2: footprint (none) -> Capacitors_THT:C_Axial_L5.1mm_D3.1mm_P7.50mm_Horizontal
- P4: footprint (none) -> Pin_Headers:Pin_Header_Straight_1x03_Pitch2.54mm
- P5: footprint (none) -> Pin_Headers:Pin_Header_Straight_1x02_Pitch2.54mm
- R3: footprint (none) -> Resistors_THT:R_Axial_DIN0207_L6.3mm_D2.5mm_P10.16mm_Horizontal
- R4: footprint (none) -> hv:R_Axial_DIN0309_L9.0mm_D3.2mm_P12.70mm_Horizontal_Thick
- U1, U5: footprint (none) -> Housings_DIP:DIP-16_W7.62mm
- U6: footprint (none) -> hv:IN12
Changed lines of the file:
@@
 F 0 "U1" H 3950 3400 50  0000 C CNN
 F 1 "4518" H 4100 2600 50  0000 C CNN
-F 2 "" H 3900 2950 60  0001 C CNN
+F 2 "Housings_DIP:DIP-16_W7.62mm" H 3900 2950 60  0001 C CNN
 F 3 "" H 3900 2950 60  0001 C CNN
 	2    3900 2950
@@
 F 0 "U5" H 6800 3200 60  0000 C CNN
 F 1 "K155ID1" H 6850 3300 60  0000 C CNN
-F 2 "" H 6800 3350 60  0001 C CNN
+F 2 "Housings_DIP:DIP-16_W7.62mm" H 6800 3350 60  0001 C CNN
 F 3 "" H 6800 3350 60  0001 C CNN
 	1    6800 3350
@@
 F 0 "U6" H 9000 4650 60  0000 C CNN
 F 1 "IN-12" H 9000 4750 60  0000 C CNN
-F 2 "" H 9000 4750 60  0001 C CNN
+F 2 "hv:IN12" H 9000 4750 60  0001 C CNN
 F 3 "" H 9000 4750 60  0001 C CNN
 	1    9000 4750
@@
 F 0 "R4" V 8380 5900 50  0000 C CNN
 F 1 "33K" V 8300 5900 50  0000 C CNN
-F 2 "" V 8230 5900 50  0000 C CNN
+F 2 "hv:R_Axial_DIN0309_L9.0mm_D3.2mm_P12.70mm_Horizontal_Thick" V 8230 5900 50  0001 C CNN
 F 3 "" H 8300 5900 50  0000 C CNN
 	1    8300 5900
@@
 F 0 "P4" H 2200 3850 50  0000 C CNN
 F 1 "CONN_01X03" V 2300 3650 50  0000 C CNN
-F 2 "" H 2200 3650 50  0000 C CNN
+F 2 "Pin_Headers:Pin_Header_Straight_1x03_Pitch2.54mm" H 2200 3650 50  0001 C CNN
 F 3 "" H 2200 3650 50  0000 C CNN
 	1    2200 3650
@@
 F 0 "P5" H 2950 4000 50  0000 C CNN
 F 1 "CONN_01X02" V 3050 3850 50  0000 C CNN
-F 2 "" H 2950 3850 50  0000 C CNN
+F 2 "Pin_Headers:Pin_Header_Straight_1x02_Pitch2.54mm" H 2950 3850 50  0001 C CNN
 F 3 "" H 2950 3850 50  0000 C CNN
 	1    2950 3850
@@
 F 0 "R3" V 2530 3250 50  0000 C CNN
 F 1 "1K" V 2450 3250 50  0000 C CNN
-F 2 "" V 2380 3250 50  0000 C CNN
+F 2 "Resistors_THT:R_Axial_DIN0207_L6.3mm_D2.5mm_P10.16mm_Horizontal" V 2380 3250 50  0001 C CNN
 F 3 "" H 2450 3250 50  0000 C CNN
 	1    2450 3250
@@
 F 0 "C2" H 2625 3950 50  0000 L CNN
 F 1 "0.1uF" H 2400 3750 50  0000 L CNN
-F 2 "" H 2638 3700 50  0000 C CNN
+F 2 "Capacitors_THT:C_Axial_L5.1mm_D3.1mm_P7.50mm_Horizontal" H 2638 3700 50  0001 C CNN
 F 3 "" H 2600 3850 50  0000 C CNN
 	1    2600 3850
