File: nixie_supply/nixie_supply.sch (KiCad schematic (older format))
At the start: 2 parts

Commit message: minor cleanups
Parts:
- gave numbers to parts that had none: 2
Changed lines of the file:
@@
 $EndSheet
 $Comp
-L CONN_01X02 P?
+L CONN_01X02 P1
 U 1 1 59110A3C
 P 2850 3000
-F 0 "P?" H 2850 3150 50  0000 C CNN
+F 0 "P1" H 2850 3150 50  0000 C CNN
 F 1 "CONN_01X02" V 2950 3000 50  0000 C CNN
 F 2 "" H 2850 3000 50  0000 C CNN
@@
 $EndComp
 $Comp
-L CONN_01X04 P?
+L CONN_01X04 P2
 U 1 1 59112A3C
 P 8650 3900
-F 0 "P?" H 8650 4150 50  0000 C CNN
+F 0 "P2" H 8650 4150 50  0000 C CNN
 F 1 "CONN_01X04" V 8750 3900 50  0000 C CNN
 F 2 "" H 8650 3900 50  0000 C CNN
@@
 	2650 2550 3500 2550
 Wire Wire Line
-	2650 3050 2550 3050
+	2550 3050 2650 3050
 Wire Wire Line
-	2550 3050 2550 2400
-Wire Wire Line
-	2550 2400 3500 2400
+	2550 2250 2550 3050
 Wire Wire Line
 	6350 4200 8450 4200
@@
 	5050 4500 5050 2850
 Connection ~ 5050 2850
+$Comp
+L PWR_FLAG #FLG01
+U 1 1 59137EF8
+P 2550 2250
+F 0 "#FLG01" H 2550 2345 50  0001 C CNN
+F 1 "PWR_FLAG" H 2550 2430 50  0000 C CNN
+F 2 "" H 2550 2250 50  0000 C CNN
+F 3 "" H 2550 2250 50  0000 C CNN
+	1    2550 2250
+	1    0    0    -1
+$EndComp
+$Comp
+L PWR_FLAG #FLG02
+U 1 1 59137F64
+P 3050 2250
+F 0 "#FLG02" H 3050 2345 50  0001 C CNN
+F 1 "PWR_FLAG" H 3050 2430 50  0000 C CNN
+F 2 "" H 3050 2250 50  0000 C CNN
+F 3 "" H 3050 2250 50  0000 C CNN
+	1    3050 2250
+	1    0    0    -1
+$EndComp
+Connection ~ 2550 2400
+Wire Wire Line
+	2550 2400 3500 2400
+Wire Wire Line
+	3050 2250 3050 2550
+Connection ~ 3050 2550
 $EndSCHEMATC

Commit message: Footprint associations
Parts:
- P1: footprint (none) -> Pin_Headers:Pin_Header_Straight_1x02_Pitch2.54mm
- P2: footprint (none) -> Pin_Headers:Pin_Header_Straight_1x04_Pitch2.54mm
Changed lines of the file:
@@
 F 0 "P1" H 2850 3150 50  0000 C CNN
 F 1 "CONN_01X02" V 2950 3000 50  0000 C CNN
-F 2 "" H 2850 3000 50  0000 C CNN
+F 2 "Pin_Headers:Pin_Header_Straight_1x02_Pitch2.54mm" H 2850 3000 50  0001 C CNN
 F 3 "" H 2850 3000 50  0000 C CNN
 	1    2850 3000
@@
 F 0 "P2" H 8650 4150 50  0000 C CNN
 F 1 "CONN_01X04" V 8750 3900 50  0000 C CNN
-F 2 "" H 8650 3900 50  0000 C CNN
+F 2 "Pin_Headers:Pin_Header_Straight_1x04_Pitch2.54mm" H 8650 3900 50  0001 C CNN
 F 3 "" H 8650 3900 50  0000 C CNN
 	1    8650 3900

Commit message: Supply board mk2: reduced time base noise, upped some clearances, added ground plane
Parts:
- removed P2: CONN_01X04, Pin_Headers:Pin_Header_Straight_1x04_Pitch2.54mm, symbol CONN_01X04
- added J1: CONN_01X01, Pin_Headers:Pin_Header_Straight_1x01_Pitch2.54mm, symbol CONN_01X01
- added J2: CONN_01X03, Pin_Headers:Pin_Header_Straight_1x03_Pitch2.54mm, symbol CONN_01X03
Connections:
- net High Voltage PSU/220V: now also J1.1 (P1)
- net High Voltage PSU/5V: now also J2.1 (P1)
- net High Voltage PSU/GND: now also J2.2 (P2)
- net PPS/CLK_OUT: now also J2.3 (P3)
- net PPS/-12VAC renamed PSU/-12VAC
Changed lines of the file:
@@
 F2 "5V" I L 5350 4050 60
 F3 "+12VAC" I L 5350 4200 60
-F4 "-12VAC" I L 5350 4350 60
-F5 "CLK_OUT" I R 6350 4200 60
-F6 "GND" I L 5350 4500 60
+F4 "CLK_OUT" I R 6350 4200 60
+F5 "GND" I L 5350 4500 60
 $EndSheet
 $Comp
@@
 F 3 "" H 2850 3000 50  0000 C CNN
 	1    2850 3000
-	1    0    0    -1
-$EndComp
-$Comp
-L CONN_01X04 P2
-U 1 1 59112A3C
-P 8650 3900
-F 0 "P2" H 8650 4150 50  0000 C CNN
-F 1 "CONN_01X04" V 8750 3900 50  0000 C CNN
-F 2 "Pin_Headers:Pin_Header_Straight_1x04_Pitch2.54mm" H 8650 3900 50  0001 C CNN
-F 3 "" H 8650 3900 50  0000 C CNN
-	1    8650 3900
 	1    0    0    -1
 $EndComp
@@
 	7900 3750 7900 3950
 Wire Wire Line
-	7900 3950 8450 3950
+	7900 3950 8550 3950
 Wire Wire Line
 	4900 2650 6200 2650
@@
 	8050 3650 8050 3850
 Wire Wire Line
-	8050 3850 8450 3850
-Wire Wire Line
-	7950 3100 8200 3100
-Wire Wire Line
-	8200 3100 8200 3750
-Wire Wire Line
-	8200 3750 8450 3750
+	8050 3850 8550 3850
 Wire Wire Line
 	6450 2700 5750 2700
@@
 	3400 4200 3400 2400
 Connection ~ 3400 2400
-Wire Wire Line
-	5350 4350 3200 4350
-Wire Wire Line
-	3200 4350 3200 2550
-Connection ~ 3200 2550
 Wire Wire Line
 	5050 4500 5050 2850
@@
 	3050 2250 3050 2550
 Connection ~ 3050 2550
+$Comp
+L CONN_01X03 J2
+U 1 1 598577B3
+P 8750 3950
+F 0 "J2" H 8750 4150 50  0000 C CNN
+F 1 "CONN_01X03" V 8850 3950 50  0000 C CNN
+F 2 "Pin_Headers:Pin_Header_Straight_1x03_Pitch2.54mm" H 8750 3950 50  0001 C CNN
+F 3 "" H 8750 3950 50  0001 C CNN
+	1    8750 3950
+	1    0    0    -1
+$EndComp
+$Comp
+L CONN_01X01 J1
+U 1 1 59857838
+P 8800 3100
+F 0 "J1" H 8800 3200 50  0000 C CNN
+F 1 "CONN_01X01" V 8900 3100 50  0000 C CNN
+F 2 "Pin_Headers:Pin_Header_Straight_1x01_Pitch2.54mm" H 8800 3100 50  0001 C CNN
+F 3 "" H 8800 3100 50  0001 C CNN
+	1    8800 3100
+	1    0    0    -1
+$EndComp
+Wire Wire Line
+	8450 4050 8550 4050
+Wire Wire Line
+	7950 3100 8600 3100
 $EndSCHEMATC

Commit message: Added more noise reduction to clock signal, added top ground plane
Connections:
- net High Voltage PSU/220V renamed High Voltage PSU/240V
Changed lines of the file:
@@
 F1 "high_voltage_power.sch" 60
 F2 "5V" I L 6450 2400 60
-F3 "220V" I R 7950 3100 60
-F4 "GND" I L 6450 2700 60
-F5 "12V" I L 6450 2850 60
+F3 "GND" I L 6450 2700 60
+F4 "12V" I L 6450 2850 60
+F5 "240V" I R 7950 3100 60
 $EndSheet
 $Sheet
