File: nixie_supply/nixie_supply.kicad_pcb (KiCad board)
At the start: 2 copper layers, 66 x 50.8 mm, 30 parts, among them J1 CONN_01X01, J2 CONN_01X03, J3 CONN_01X03, P1 CONN_01X02, Q1 FQPF4N90CT, U1 LM741, U2 4047, U3 7805, U4 LM555N, U5 4518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

Commit message: Overhaul of clock board. Fixed hour digits, added more noise immunity, reduced height
Changed lines of the file:
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@@
     (links 68)
     (no_connects 0)
-    (area 81.204999 83.744999 147.395001 134.695001)
+    (area 78.235 82.734999 148.405001 136.955)
     (thickness 1.6)
     (drawings 4)
@@
     (visible_elements 7FFFFFFF)
     (pcbplotparams
-      (layerselection 0x010f0_80000001)
+      (layerselection 0x00020_00000000)
       (usegerberextensions false)
       (excludeedgelayer true)
@@
       (drillshape 0)
       (scaleselection 1)
-      (outputdirectory gerber_files/))
+      (outputdirectory nixie_supply_gerber_files_0.2/))
   )
   (net 0 "")
@@
     (descr "module 1 pin (ou trou mecanique de percage)")
     (tags DEV)
-    (fp_text reference REF** (at 0 -3.048) (layer F.SilkS)
+    (fp_text reference REF** (at -5.08 -1.27) (layer F.SilkS)
       (effects (font (size 1 1) (thickness 0.15)))
     )
@@
     (descr "module 1 pin (ou trou mecanique de percage)")
     (tags DEV)
-    (fp_text reference REF** (at 0 -3.048) (layer F.SilkS)
-      (effects (font (size 1 1) (thickness 0.15)))
-    )
+    (fp_text reference REF** (at 5.08 -1.27) (layer F.SilkS)
+      (effects (font (size 1 1) (thickness 0.15)))
+    )
